File: aliasing.kicad_pcb (KiCad board)
At the start: 2 copper layers, 50 x 57 mm, 18 parts, among them J1001 Conn_Coaxial, J1002 Conn_Coaxial, J1003 Conn_Coaxial, J1004 Conn_Coaxial, J1005 Conn_Coaxial, J1006 Conn_Coaxial, J1007 Conn_01x01_Female, J1008 Conn_01x01_Female, J1009 Conn_01x01_Female, J1010 Conn_01x01_Female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

Commit message: TLV diodes added, new gerber, minor modif.
Parts:
- removed REF**: KiCad-Logo2_6mm_SilkScreen, Symbol:KiCad-Logo2_6mm_SilkScreen
- removed REF**: OSHW-Logo2_7.3x6mm_SilkScreen, Symbol:OSHW-Logo2_7.3x6mm_SilkScreen
- added D1: CD05_SOD323-T05, Diode_SMD:D_SOD-323, B.Cu at (180.0, 67.0)
- added D2: CD05_SOD323-T05, Diode_SMD:D_SOD-323, B.Cu at (180.0, 52.0)
